File: pcb/ble-receiver.kicad_pcb (KiCad board)
At the start: 2 copper layers, 30.2 x 18.8 mm, 33 parts, among them J1 Conn_Coaxial, J2 Conn_01x04, J3 CH1, J4 CH2, J5 CH3, J6 CH4, J7 CH5, U1 TPS62203DBV, U2 nRF52832-QFxx, Y1 32Mhz

Commit message: bump kicad version
Parts:
- J2, J3, J4, J5, J6, J7: moved to B.Cu
- turned J2 to 90 degrees
- turned J3 to 90 degrees
- turned J4 to 90 degrees
- turned J5 to 90 degrees
- turned J6 to 90 degrees
- turned J7 to 90 degrees
