File: pcb/ble-receiver.kicad_sch (KiCad schematic)
At the start: 32 parts, among them J1 Conn_Coaxial, J2 Conn_01x04, J3 CH1, J4 CH2, J5 CH3, J6 CH4, J7 CH5, U1 TPS62203DBV, U2 nRF52832-QFxx, Y1 32Mhz

Commit message: bump kicad version
Changed lines of the file:
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@@
 (kicad_sch
-	(version 20231120)
+	(version 20250114)
 	(generator "eeschema")
-	(generator_version "8.0")
+	(generator_version "9.0")
 	(paper "A4")
 	(title_block
@@
 	(label "BATTERY_LEVEL"
 		(at 54.61 80.01 0)
-		(fields_autoplaced yes)
 		(effects
 			(font
@@
 	(label "SWDIO"
 		(at 95.25 161.29 0)
-		(fields_autoplaced yes)
 		(effects
 			(font
@@
 	(label "SWDCLK"
 		(at 95.25 158.75 0)
-		(fields_autoplaced yes)
 		(effects
 			(font
@@
 	(label "DCDC_FB"
 		(at 109.22 44.45 0)
-		(fields_autoplaced yes)
 		(effects
 			(font
@@
 	(label "CH2"
 		(at 161.29 92.71 0)
-		(fields_autoplaced yes)
 		(effects
 			(font
@@
 	(label "CH5"
 		(at 161.29 100.33 0)
-		(fields_autoplaced yes)
 		(effects
 			(font
@@
 	(label "CH1"
 		(at 161.29 90.17 0)
-		(fields_autoplaced yes)
 		(effects
 			(font
@@
 	(label "CH3"
 		(at 161.29 95.25 0)
-		(fields_autoplaced yes)
 		(effects
 			(font
@@
 	(label "DCDC_OUT"
 		(at 110.49 39.37 90)
-		(fields_autoplaced yes)
 		(effects
 			(font
@@
 	(label "STATUS_LED"
 		(at 161.29 118.11 0)
-		(fields_autoplaced yes)
 		(effects
 			(font
@@
 	(label "BATTERY_LEVEL"
 		(at 161.29 102.87 0)
-		(fields_autoplaced yes)
 		(effects
 			(font
@@
 	(label "DCDC_EN"
 		(at 87.63 41.91 180)
-		(fields_autoplaced yes)
 		(effects
 			(font
@@
 	(label "CH4"
 		(at 161.29 97.79 0)
-		(fields_autoplaced yes)
 		(effects
 			(font
@@
 		)
 	)
+	(embedded_fonts no)
 )
